File: KiCAD/WULP/_autosave-Power.sch (KiCad schematic (older format))
At the start: 3 parts, among them U1 AMS1117-3.3

Commit message: power + micro
Parts:
- added J?: USB_B_Micro, Connector_USB:USB_Micro-B_Molex_47346-0001, symbol Connector:USB_B_Micro
- added U?: USBLC6-2SC6, Package_TO_SOT_SMD:SOT-23-6, symbol Power_Protection:USBLC6-2SC6
- C1: value C_Small -> 100nF
- C2: value C_Small -> 22pF
Connections:
- net +5V: now also J?.1 (VBUS), U?.5 (VBUS)
- net GND: now also J?.5 (GND), U?.2 (GND)
- new net USB_CONN_D+: J?.3 (D+), U?.3 (I/O2)
- new net USB_CONN_D-: J?.2 (D-), U?.1 (I/O1)
- new net USB_D+: U?.4 (I/O2)
- new net USB_D-: U?.6 (I/O1)
- no-connect marks 0 -> 2
Other:
- moved on the sheet: C1, C2, U1
Changed lines of the file:
@@
 $Descr A4 11693 8268
 encoding utf-8
-Sheet 2 2
+Sheet 2 3
 Title ""
 Date ""
@@
 L Regulator_Linear:AMS1117-3.3 U1
 U 1 1 61B2636E
-P 3450 1750
-F 0 "U1" H 3450 1992 50  0000 C CNN
-F 1 "AMS1117-3.3" H 3450 1901 50  0000 C CNN
-F 2 "Package_TO_SOT_SMD:SOT-223-3_TabPin2" H 3450 1950 50  0001 C CNN
-F 3 "http://www.advanced-monolithic.com/pdf/ds1117.pdf" H 3550 1500 50  0001 C CNN
-F 4 "C6186" H 3450 1750 50  0001 C CNN "LCSC"
-	1    3450 1750
+P 8000 3600
+F 0 "U1" H 8000 3842 50  0000 C CNN
+F 1 "AMS1117-3.3" H 8000 3751 50  0000 C CNN
+F 2 "Package_TO_SOT_SMD:SOT-223-3_TabPin2" H 8000 3800 50  0001 C CNN
+F 3 "http://www.advanced-monolithic.com/pdf/ds1117.pdf" H 8100 3350 50  0001 C CNN
+F 4 "C6186" H 8000 3600 50  0001 C CNN "LCSC"
+	1    8000 3600
 	1    0    0    -1
 $EndComp
@@
 L Device:C_Small C1
 U 1 1 61B2801B
-P 2650 1900
-F 0 "C1" H 2742 1946 50  0000 L CNN
-F 1 "C_Small" H 2742 1855 50  0000 L CNN
-F 2 "" H 2650 1900 50  0001 C CNN
-F 3 "~" H 2650 1900 50  0001 C CNN
-	1    2650 1900
+P 7200 3750
+F 0 "C1" H 7292 3796 50  0000 L CNN
+F 1 "100nF" H 7292 3705 50  0000 L CNN
+F 2 "" H 7200 3750 50  0001 C CNN
+F 3 "~" H 7200 3750 50  0001 C CNN
+	1    7200 3750
 	1    0    0    -1
 $EndComp
@@
 L Device:C_Small C2
 U 1 1 61B28A2B
-P 4200 1900
-F 0 "C2" H 4292 1946 50  0000 L CNN
-F 1 "C_Small" H 4292 1855 50  0000 L CNN
-F 2 "" H 4200 1900 50  0001 C CNN
-F 3 "~" H 4200 1900 50  0001 C CNN
-	1    4200 1900
+P 8750 3750
+F 0 "C2" H 8842 3796 50  0000 L CNN
+F 1 "22pF" H 8842 3705 50  0000 L CNN
+F 2 "" H 8750 3750 50  0001 C CNN
+F 3 "~" H 8750 3750 50  0001 C CNN
+	1    8750 3750
 	1    0    0    -1
 $EndComp
@@
 L power:GND #PWR0101
 U 1 1 61B29583
-P 3450 2100
-F 0 "#PWR0101" H 3450 1850 50  0001 C CNN
-F 1 "GND" H 3455 1927 50  0000 C CNN
-F 2 "" H 3450 2100 50  0001 C CNN
-F 3 "" H 3450 2100 50  0001 C CNN
-	1    3450 2100
+P 8000 3950
+F 0 "#PWR0101" H 8000 3700 50  0001 C CNN
+F 1 "GND" H 8005 3777 50  0000 C CNN
+F 2 "" H 8000 3950 50  0001 C CNN
+F 3 "" H 8000 3950 50  0001 C CNN
+	1    8000 3950
 	1    0    0    -1
 $EndComp
@@
 L power:GND #PWR0102
 U 1 1 61B29A1A
-P 2650 2050
-F 0 "#PWR0102" H 2650 1800 50  0001 C CNN
-F 1 "GND" H 2655 1877 50  0000 C CNN
-F 2 "" H 2650 2050 50  0001 C CNN
-F 3 "" H 2650 2050 50  0001 C CNN
-	1    2650 2050
+P 7200 3900
+F 0 "#PWR0102" H 7200 3650 50  0001 C CNN
+F 1 "GND" H 7205 3727 50  0000 C CNN
+F 2 "" H 7200 3900 50  0001 C CNN
+F 3 "" H 7200 3900 50  0001 C CNN
+	1    7200 3900
 	1    0    0    -1
 $EndComp
@@
 L power:GND #PWR0103
 U 1 1 61B29D60
-P 4200 2050
-F 0 "#PWR0103" H 4200 1800 50  0001 C CNN
-F 1 "GND" H 4205 1877 50  0000 C CNN
-F 2 "" H 4200 2050 50  0001 C CNN
-F 3 "" H 4200 2050 50  0001 C CNN
-	1    4200 2050
+P 8750 3900
+F 0 "#PWR0103" H 8750 3650 50  0001 C CNN
+F 1 "GND" H 8755 3727 50  0000 C CNN
+F 2 "" H 8750 3900 50  0001 C CNN
+F 3 "" H 8750 3900 50  0001 C CNN
+	1    8750 3900
 	1    0    0    -1
 $EndComp
@@
 L power:+3.3V #PWR0104
 U 1 1 61B2AD40
-P 4550 1700
-F 0 "#PWR0104" H 4550 1550 50  0001 C CNN
-F 1 "+3.3V" H 4565 1873 50  0000 C CNN
-F 2 "" H 4550 1700 50  0001 C CNN
-F 3 "" H 4550 1700 50  0001 C CNN
-	1    4550 1700
-	1    0    0    -1
-$EndComp
-Wire Wire Line
-	2650 1800 2650 1750
-Wire Wire Line
-	2650 1750 3150 1750
-Wire Wire Line
-	3750 1750 4200 1750
-Wire Wire Line
-	4200 1750 4200 1800
-Wire Wire Line
-	4200 1750 4550 1750
-Wire Wire Line
-	4550 1750 4550 1700
-Connection ~ 4200 1750
-Wire Wire Line
-	4200 2050 4200 2000
-Wire Wire Line
-	3450 2050 3450 2100
-Wire Wire Line
-	2650 2050 2650 2000
-Connection ~ 2650 1750
-Wire Wire Line
-	2300 1750 2650 1750
-Wire Wire Line
-	2300 1700 2300 1750
+P 9100 3550
+F 0 "#PWR0104" H 9100 3400 50  0001 C CNN
+F 1 "+3.3V" H 9115 3723 50  0000 C CNN
+F 2 "" H 9100 3550 50  0001 C CNN
+F 3 "" H 9100 3550 50  0001 C CNN
+	1    9100 3550
+	1    0    0    -1
+$EndComp
+Wire Wire Line
+	7200 3650 7200 3600
+Wire Wire Line
+	7200 3600 7700 3600
+Wire Wire Line
+	8300 3600 8750 3600
+Wire Wire Line
+	8750 3600 8750 3650
+Wire Wire Line
+	8750 3600 9100 3600
+Wire Wire Line
+	9100 3600 9100 3550
+Connection ~ 8750 3600
+Wire Wire Line
+	8750 3900 8750 3850
+Wire Wire Line
+	8000 3900 8000 3950
+Wire Wire Line
+	7200 3900 7200 3850
+Connection ~ 7200 3600
+Wire Wire Line
+	6850 3600 7200 3600
+Wire Wire Line
+	6850 3550 6850 3600
 $Comp
 L power:+5V #PWR0105
 U 1 1 61B2A181
-P 2300 1700
-F 0 "#PWR0105" H 2300 1550 50  0001 C CNN
-F 1 "+5V" H 2315 1873 50  0000 C CNN
-F 2 "" H 2300 1700 50  0001 C CNN
-F 3 "" H 2300 1700 50  0001 C CNN
-	1    2300 1700
-	1    0    0    -1
-$EndComp
+P 6850 3550
+F 0 "#PWR0105" H 6850 3400 50  0001 C CNN
+F 1 "+5V" H 6865 3723 50  0000 C CNN
+F 2 "" H 6850 3550 50  0001 C CNN
+F 3 "" H 6850 3550 50  0001 C CNN
+	1    6850 3550
+	1    0    0    -1
+$EndComp
+$Comp
+L Connector:USB_B_Micro J?
+U 1 1 61B3179E
+P 2500 3750
+F 0 "J?" H 2557 4217 50  0000 C CNN
+F 1 "USB_B_Micro" H 2557 4126 50  0000 C CNN
+F 2 "Connector_USB:USB_Micro-B_Molex_47346-0001" H 2650 3700 50  0001 C CNN
+F 3 "~" H 2650 3700 50  0001 C CNN
+F 4 "C132560" H 2500 3750 50  0001 C CNN "LCSC"
+	1    2500 3750
+	1    0    0    -1
+$EndComp
+$Comp
+L power:+5V #PWR?
+U 1 1 61B33641
+P 3050 3450
+F 0 "#PWR?" H 3050 3300 50  0001 C CNN
+F 1 "+5V" H 3065 3623 50  0000 C CNN
+F 2 "" H 3050 3450 50  0001 C CNN
+F 3 "" H 3050 3450 50  0001 C CNN
+	1    3050 3450
+	1    0    0    -1
+$EndComp
+Text GLabel 3050 3750 2    50   Input ~ 0
+USB_CONN_D+
+Text GLabel 3050 3850 2    50   Input ~ 0
+USB_CONN_D-
+Wire Wire Line
+	2800 3750 3050 3750
+Wire Wire Line
+	2800 3850 3050 3850
+Wire Wire Line
+	2800 3550 3050 3550
+Wire Wire Line
+	3050 3550 3050 3450
+$Comp
+L power:GND #PWR?
+U 1 1 61B34BC4
+P 2500 4200
+F 0 "#PWR?" H 2500 3950 50  0001 C CNN
+F 1 "GND" H 2505 4027 50  0000 C CNN
+F 2 "" H 2500 4200 50  0001 C CNN
+F 3 "" H 2500 4200 50  0001 C CNN
+	1    2500 4200
+	1    0    0    -1
+$EndComp
+Wire Wire Line
+	2500 4150 2500 4200
+NoConn ~ 2400 4150
+NoConn ~ 2800 3950
+$Comp
+L Power_Protection:USBLC6-2SC6 U?
+U 1 1 61B41C1F
+P 5150 3800
+F 0 "U?" H 5450 4300 50  0000 C CNN
+F 1 "USBLC6-2SC6" H 5450 4200 50  0000 C CNN
+F 2 "Package_TO_SOT_SMD:SOT-23-6" H 5150 3300 50  0001 C CNN
+F 3 "https://www.st.com/resource/en/datasheet/usblc6-2.pdf" H 5350 4150 50  0001 C CNN
+F 4 "C2827654" H 5150 3800 50  0001 C CNN "LCSC"
+	1    5150 3800
+	1    0    0    -1
+$EndComp
+Text GLabel 5650 3900 2    50   Input ~ 0
+USB_CONN_D+
+Text GLabel 4650 3900 0    50   Input ~ 0
+USB_CONN_D-
+Text GLabel 4650 3700 0    50   Input ~ 0
+USB_D-
+Text GLabel 5650 3700 2    50   Input ~ 0
+USB_D+
+Wire Wire Line
+	5550 3700 5650 3700
+Wire Wire Line
+	5650 3900 5550 3900
+Wire Wire Line
+	4750 3700 4650 3700
+Wire Wire Line
+	4750 3900 4650 3900
+$Comp
+L power:+5V #PWR?
+U 1 1 61B469CF
+P 5150 3300
+F 0 "#PWR?" H 5150 3150 50  0001 C CNN
+F 1 "+5V" H 5165 3473 50  0000 C CNN
+F 2 "" H 5150 3300 50  0001 C CNN
+F 3 "" H 5150 3300 50  0001 C CNN
+	1    5150 3300
+	1    0    0    -1
+$EndComp
+Wire Wire Line
+	5150 3400 5150 3300
+$Comp
+L power:GND #PWR?
+U 1 1 61B47359
+P 5150 4250
+F 0 "#PWR?" H 5150 4000 50  0001 C CNN
+F 1 "GND" H 5155 4077 50  0000 C CNN
+F 2 "" H 5150 4250 50  0001 C CNN
+F 3 "" H 5150 4250 50  0001 C CNN
+	1    5150 4250
+	1    0    0    -1
+$EndComp
+Wire Wire Line
+	5150 4250 5150 4200
 $EndSCHEMATC
