File: KiCAD/WULP/_autosave-WULP.sch (KiCad schematic (older format))
At the start: 0 parts

Commit message: power + micro
Changed lines of the file:
@@
 $Descr A4 11693 8268
 encoding utf-8
-Sheet 1 2
+Sheet 1 3
 Title ""
 Date ""
@@
 F1 "Power.sch" 50
 $EndSheet
+$Sheet
+S 2050 3500 950  650
+U 61B53C83
+F0 "Microcontroller" 50
+F1 "Microcontroller.sch" 50
+$EndSheet
 $EndSCHEMATC
