File: KiCAD/WULP/Power.sch (KiCad schematic (older format))
At the start: 9 parts, among them J1 USB_B_Micro, U1 AMS1117-3.3, U2 USBLC6-2SC6

Commit message: pulled WULP to personal machine
Other:
- note added: "Find lower Q current regulator, this one is typ 5mA\n"
Changed lines of the file:
@@
 	1    0    0    -1
 $EndComp
+Text Notes 7050 3150 0    50   ~ 0
+Find lower Q current regulator, this one is typ 5mA\n
 $EndSCHEMATC
